File: hardware/openLager.kicad_pcb (KiCad board)
At the start: 4 copper layers, 15.2 x 19 mm, 30 parts, among them J1 CONN_01X06, J2 DM3CS-SF, U1 STM32F411CEUx, U2 SPX3819M5-L-3-3, Y1 CSTCE8M00G15L99

Commit message: Change /NRST from pin to TP
Parts:
- TP1: footprint openLagerFootprints:Socket_Strip_Straight_1x01 -> openLagerFootprints:TP
- moved TP1 5.75 mm to (191.1, 106.0)
Routing:
- net NRST: track 12.7 -> 5.30 mm, vias 1 -> 0
- net GND: vias 12 -> 13
Other:
- board text removed: "NRST"
Changed lines of the file:
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@@
     (area 186.709267 94.1961 208.776305 121.981539)
     (thickness 1.6)
-    (drawings 13)
-    (tracks 434)
+    (drawings 12)
+    (tracks 428)
     (zones 0)
     (modules 30)
@@
       (rotate (xyz 0 0 180))
     )
-  )
-  (module openLagerFootprints:Socket_Strip_Straight_1x01 (layer F.Cu)
-    (at 191.77 111.76)
-    (descr "Through hole socket strip")
-    (tags "socket strip")
-    (fp_text reference TP1 (at -0.0635 -1.4605) (layer F.SilkS)
-      (effects (font (size 0.5 0.5) (thickness 0.125)))
-    )
-    (fp_text value TEST_1P (at 0 -3.1) (layer F.Fab) hide
-      (effects (font (size 1 1) (thickness 0.15)))
-    )
-    (fp_line (start -1.75 -1.75) (end -1.75 1.75) (layer F.CrtYd) (width 0.05))
-    (fp_line (start 1.75 -1.75) (end 1.75 1.75) (layer F.CrtYd) (width 0.05))
-    (fp_line (start -1.75 -1.75) (end 1.75 -1.75) (layer F.CrtYd) (width 0.05))
-    (fp_line (start -1.75 1.75) (end 1.75 1.75) (layer F.CrtYd) (width 0.05))
-    (pad 1 thru_hole rect (at 0 0) (size 1.7272 2.032) (drill 1.016) (layers *.Cu *.Mask F.SilkS)
-      (net 4 NRST))
   )
   (module openLagerFootprints:SOT95P280X145-5N (layer F.Cu)
@@
       (xy -1.94426 -1.037172) (xy -1.942844 -1.035594)) (layer F.SilkS) (width 0.01))
   )
+  (module openLagerFootprints:TP (layer F.Cu)
+    (at 191.135 106.045)
+    (fp_text reference TP1 (at 0 0.5) (layer F.SilkS) hide
+      (effects (font (size 1 1) (thickness 0.15)))
+    )
+    (fp_text value TEST_1P (at 0 -0.5) (layer F.Fab) hide
+      (effects (font (size 1 1) (thickness 0.15)))
+    )
+    (pad 1 thru_hole circle (at 0 0) (size 0.6858 0.6858) (drill 0.3302) (layers *.Cu *.Mask F.SilkS)
+      (net 4 NRST))
+  )
   (gr_text SI (at 204.47 112.649) (layer B.SilkS)
     (effects (font (size 0.5 0.5) (thickness 0.1)) (justify mirror))
@@
   )
   (gr_text SO (at 193.2305 112.7125) (layer B.SilkS)
-    (effects (font (size 0.5 0.5) (thickness 0.1)) (justify mirror))
-  )
-  (gr_text NRST (at 193.675 111.6965) (layer B.SilkS)
     (effects (font (size 0.5 0.5) (thickness 0.1)) (justify mirror))
   )
@@
   (segment (start 199.1868 112.1664) (end 199.1868 112.0267) (width 0.508) (layer F.Cu) (net 1))
   (segment (start 199.1868 114.0968) (end 199.39 114.3) (width 0.508) (layer F.Cu) (net 1))
+  (via (at 191.5795 112.141) (size 0.6858) (drill 0.3302) (layers F.Cu B.Cu) (net 2))
   (segment (start 197.739 111.0615) (end 196.2365 111.0615) (width 0.47625) (layer F.Cu) (net 2))
   (segment (start 196.2365 111.0615) (end 196.1515 110.9765) (width 0.47625) (layer F.Cu) (net 2))
@@
   (segment (start 192.2145 107.1245) (end 191.77 106.68) (width 0.254) (layer F.Cu) (net 3))
   (segment (start 193.675 107.1245) (end 192.2145 107.1245) (width 0.254) (layer F.Cu) (net 3))
-  (via (at 191.135 106.045) (size 0.6858) (drill 0.3302) (layers F.Cu B.Cu) (net 4))
+  (segment (start 193.3575 106.4895) (end 192.786 105.918) (width 0.1524) (layer F.Cu) (net 4))
+  (segment (start 192.786 105.918) (end 192.024 105.918) (width 0.1524) (layer F.Cu) (net 4))
+  (segment (start 192.024 105.918) (end 191.897 106.045) (width 0.1524) (layer F.Cu) (net 4))
   (segment (start 191.897 106.045) (end 191.135 106.045) (width 0.1524) (layer F.Cu) (net 4))
-  (segment (start 192.024 105.918) (end 191.897 106.045) (width 0.1524) (layer F.Cu) (net 4))
-  (segment (start 192.786 105.918) (end 192.024 105.918) (width 0.1524) (layer F.Cu) (net 4))
-  (segment (start 193.3575 106.4895) (end 192.786 105.918) (width 0.1524) (layer F.Cu) (net 4))
-  (segment (start 190.754 110.744) (end 191.77 111.76) (width 0.1524) (layer B.Cu) (net 4))
-  (segment (start 190.754 106.426) (end 190.754 110.744) (width 0.1524) (layer B.Cu) (net 4))
-  (segment (start 191.135 106.045) (end 190.754 106.426) (width 0.1524) (layer B.Cu) (net 4))
-  (segment (start 192.024 111.506) (end 191.77 111.76) (width 0.1524) (layer B.Cu) (net 4))
   (segment (start 193.363 106.4895) (end 193.363 105.7005) (width 0.1524) (layer F.Cu) (net 4))
   (segment (start 193.363 105.7005) (end 193.6535 105.41) (width 0.1524) (layer F.Cu) (net 4))
@@
   (segment (start 194.6315 104.771) (end 193.9925 105.41) (width 0.1524) (layer F.Cu) (net 4))
   (segment (start 193.9925 105.41) (end 193.6535 105.41) (width 0.1524) (layer F.Cu) (net 4))
-  (segment (start 192.3415 111.125) (end 192.3415 111.818) (width 0.1524) (layer F.Cu) (net 4))
-  (segment (start 192.278 111.0615) (end 192.3415 111.125) (width 0.1524) (layer F.Cu) (net 4))
   (segment (start 200.237 108.839) (end 200.237 108.67) (width 0.254) (layer F.Cu) (net 5))
   (segment (start 200.237 108.67) (end 200.124 108.557) (width 0.254) (layer F.Cu) (net 5))
