File: hardware/openLager.sch (KiCad schematic (older format))
At the start: 29 parts, among them J1 CONN_01X06, J2 DM3CS-SF, U1 STM32F411CEUx, U2 SPX3819M5-L-3-3, Y1 CSTCE8M00G15L99

Commit message: Change /NRST from pin to TP
Parts:
- TP1: footprint openLagerFootprints:Socket_Strip_Straight_1x01 -> openLagerFootprints:TP
Changed lines of the file:
@@
 F 0 "TP1" H 13750 7600 50  0000 C CNN
 F 1 "TEST_1P" H 13750 7600 50  0001 C CNN
-F 2 "openLagerFootprints:Socket_Strip_Straight_1x01" H 13950 7400 50  0001 C CNN
+F 2 "openLagerFootprints:TP" H 13950 7400 50  0001 C CNN
 F 3 "DNP" H 13950 7400 50  0001 C CNN
 F 4 "DNP" H 13750 7400 60  0001 C CNN "Mfg Name"
